Commit message: Add lidar to husky rover

File: husky_description/urdf/husky.urdf.xacro (robot description, xacro)
@@ -33,4 +33,6 @@
   <xacro:arg name="robot_namespace" default="/" />
   <xacro:arg name="urdf_extras" default="$(find husky_description)/urdf/accessories/zed2_setup.urdf.xacro" />
+  <!-- OS1 Lidar !-->
+  <xacro:arg name="urdf_extras_lidar" default="$(find ouster_description)/urdf/OS1-64.urdf.xacro" />
   <!-- Included URDF/XACRO Files -->
   <xacro:include filename="$(find husky_description)/urdf/decorations.urdf.xacro" />
@@ -183,3 +185,7 @@
   <!-- Optional custom includes. -->
   <xacro:include filename="$(arg urdf_extras)" />
+  <xacro:include filename="$(arg urdf_extras_lidar)" />
+  <OS1-64 parent="base_link" name="os1_sensor" hz="10" samples="220">
+    <origin xyz="0 0 0.5" rpy="0 0 0" />
+  </OS1-64>
 </robot>

Commit message: Add bowler hat

File: husky_description/urdf/husky.urdf.xacro (robot description, xacro)
@@ -102,4 +102,26 @@
   <gazebo reference="imu_link">
   </gazebo>
+  <link name="bowler_link">
+    <visual>
+      <geometry>
+        <mesh filename="$(find husky_description)/meshes/red_bowler.dae" />
+      </geometry>
+    </visual>
+    <collision>
+      <origin xyz="0 0 0.07" rpy="0 0 0" />
+      <geometry>
+        <box size="0.32 0.25 0.14" rpy="0 0 0"/>
+      </geometry>
+    </collision>
+    <inertial>
+      <mass value="30"/>
+      <inertia ixx="0.4" ixy="0.0" ixz="0.0" iyy="0.4" iyz="0.0" izz="0.2"/>
+    </inertial>
+  </link>
+  <joint name="bowler_joint" type="fixed">
+    <parent link="top_plate_link" />
+    <child link="bowler_link" />
+    <origin xyz="0.02 0.2 0" rpy="0 0 0.5" />
+  </joint>
   <!-- Husky wheel macros -->
   <xacro:husky_wheel wheel_prefix="front_left">
